Commit message: works: ros2 launch ros2_control_demo_example_3 rrbot_system_multi_interface.launch.py robot_controller:=joint_trajectory_controller

File: example_3/description/ros2_control/rrbot_system_multi_interface.ros2_control.xacro (robot description, xacro)
@@ -1,17 +1,22 @@
 <?xml version="1.0"?>
 <robot xmlns:xacro="http://www.ros.org/wiki/xacro">
-  <xacro:macro name="rrbot_system_multi_interface" params="name prefix use_mock_hardware:=^|true mock_sensor_commands:=^|false slowdown:=2.0">
+  <xacro:macro name="rrbot_system_multi_interface" params="name prefix use_sim:=^|false use_mock_hardware:=^|true mock_sensor_commands:=^|false slowdown:=2.0">
     <ros2_control name="${name}" type="system">
       <hardware>
-        <xacro:if value="${use_mock_hardware}">
-          <plugin>mock_components/GenericSystem</plugin>
-          <param name="mock_sensor_commands">${mock_sensor_commands}</param>
-          <param name="state_following_offset">0.0</param>
+        <xacro:if value="$(arg use_sim)">
+          <plugin>gazebo_ros2_control/GazeboSystem</plugin>
         </xacro:if>
-        <xacro:unless value="${use_mock_hardware}">
-          <plugin>ros2_control_demo_example_3/RRBotSystemMultiInterfaceHardware</plugin>
-          <param name="example_param_hw_start_duration_sec">0.0</param>
-          <param name="example_param_hw_stop_duration_sec">3.0</param>
-          <param name="example_param_hw_slowdown">${slowdown}</param>
+        <xacro:unless value="$(arg use_sim)">
+          <xacro:if value="${use_mock_hardware}">
+            <plugin>mock_components/GenericSystem</plugin>
+            <param name="mock_sensor_commands">${mock_sensor_commands}</param>
+            <param name="state_following_offset">0.0</param>
+          </xacro:if>
+          <xacro:unless value="${use_mock_hardware}">
+            <plugin>ros2_control_demo_example_3/RRBotSystemMultiInterfaceHardware</plugin>
+            <param name="example_param_hw_start_duration_sec">0.0</param>
+            <param name="example_param_hw_stop_duration_sec">3.0</param>
+            <param name="example_param_hw_slowdown">${slowdown}</param>
+          </xacro:unless>
         </xacro:unless>
       </hardware>
@@ -29,7 +34,12 @@
           <param name="max">1</param>
         </command_interface>
+        <command_interface name="effort">
+          <param name="min">-1</param>
+          <param name="max">1</param>
+        </command_interface>
         <state_interface name="position"/>
         <state_interface name="velocity"/>
         <state_interface name="acceleration"/>
+        <state_interface name="effort"/>
       </joint>
       <joint name="${prefix}joint2">
@@ -46,7 +56,12 @@
           <param name="max">1</param>
         </command_interface>
+        <command_interface name="effort">
+          <param name="min">-1</param>
+          <param name="max">1</param>
+        </command_interface>
         <state_interface name="position"/>
         <state_interface name="velocity"/>
         <state_interface name="acceleration"/>
+        <state_interface name="effort"/>
       </joint>
     </ros2_control>

File: example_3/description/urdf/rrbot_system_multi_interface.urdf.xacro (robot description, xacro)
@@ -7,4 +7,5 @@
 <robot xmlns:xacro="http://www.ros.org/wiki/xacro" name="2dof_robot">
   <!-- Enable setting arguments from the launch file -->
+  <xacro:arg name="use_sim" default="true" />
   <xacro:arg name="use_mock_hardware" default="false" />
   <xacro:arg name="mock_sensor_commands" default="false" />
@@ -24,6 +25,13 @@
   <xacro:rrbot_system_multi_interface
     name="RRBotSystemMultiInterface" prefix="$(arg prefix)"
+    use_sim="$(arg use_sim)"
     use_mock_hardware="$(arg use_mock_hardware)"
     mock_sensor_commands="$(arg mock_sensor_commands)"
     slowdown="$(arg slowdown)" />
+  <gazebo>
+      <plugin filename="libgazebo_ros2_control.so" name="gazebo_ros2_control">
+          <parameters>$(find ros2_control_demo_example_3)/config/rrbot_multi_interface_forward_controllers.yaml
+          </parameters>
+      </plugin>
+  </gazebo>
 </robot>
